File: kicad/1541-RAMBoard2-FirstBank/1541-RAMBoard2-FirstBank.kicad_pcb (KiCad board)
At the start: 2 copper layers, 58.7 x 40.6 mm, 12 parts, among them J1 Conn_01x02_Male, U1 27C512, U2 74LS139, U3 KM62256CLP, U4_SOCKET1 27128

Commit message: revision 1.1 - no changes except messages that R/W has to be connected to RAM (U6) R/W from gate array (U10), not directly to CPU R/W
Other:
- board text added: "1541-RAMBOard][ v1.1 (c) IV 2024 Maciej Witkowiak, <ytm@elysium.pl>"
- board text added: "J1 A14 from CPU (U3) pin 24 R/~{W} from onboard RAM (U5) pin 21"
- board text removed: "1541-RAMBOard][ v1.0 (c) IV 2024 Maciej Witkowiak, <ytm@elysium.pl>"
- board text removed: "J1 A14 from CPU (U3) pin 24 R/~{W} from VIA (U6/U8) pin 22 or CPU (U3) pin 34"
Changed lines of the file:
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@@
   )
   (paper "A4")
+  (title_block
+    (title "1541-RAMBOard][")
+    (date "2024-04-20")
+    (company "YTM Enterprises")
+    (comment 1 "Maciej Witkowiak <ytm@elysium.pl>")
+  )
   (layers
     (0 "F.Cu" signal)
@@
     (effects (font (size 0.7 0.7) (thickness 0.15)) (justify left mirror))
   )
-  (gr_text "1541-RAMBOard][ v1.0\n(c) IV 2024 Maciej Witkowiak, <ytm@elysium.pl>" (at 113.792 87.63 90) (layer "B.SilkS")
+  (gr_text "1541-RAMBOard][ v1.1\n(c) IV 2024 Maciej Witkowiak, <ytm@elysium.pl>" (at 113.792 87.63 90) (layer "B.SilkS")
     (effects (font (size 0.7 0.7) (thickness 0.15)) (justify left mirror))
   )
-  (gr_text "J1\nA14 from CPU (U3) pin 24\nR/~{W} from VIA (U6/U8) pin 22 or CPU (U3) pin 34" (at 131.826 87.360143 90) (layer "B.SilkS")
+  (gr_text "J1\nA14 from CPU (U3) pin 24\nR/~{W} from onboard RAM (U5) pin 21" (at 131.826 87.360143 90) (layer "B.SilkS")
     (effects (font (size 0.7 0.7) (thickness 0.15)) (justify left mirror))
   )
